File: LibTesting.kicad_pcb (KiCad board)
At the start: 2 copper layers, 28 parts, among them IC1 LBWA1ZZ1YL, IC2 TPS23731RMTR, IC3 DART_MX93, J1 USB4200-03-A, J10 CONUFL001-SMD-T, J2 Halo_RJ45_LINKPP_LPJT96282-8C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, J3 HYBRID_T1, J4 Molex_FAKRA_73404-0812, J5 Molex_FAKRA_73404-0813, J6 Molex_FAKRA_73404-0820, J7 Molex_Mini50_12P_348260124, J8 1843800, Q1 NTMFD5C680NL, SW1 TACTA_SW_64K-F, T1 WURTH_750314782, U1 SIM68AD, U2 SCREW_MOUNTING

Commit message: ts
Other:
- board outline added: 159.8 x 96.8 mm
Changed lines of the file:
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@@
 		)
+	)
+	(gr_rect
+		(start 20 36.5)
+		(end 179.75 133.25)
+		(stroke
+			(width 0.05)
+			(type default)
+		)
+		(fill no)
+		(layer "Edge.Cuts")
 	)
 	(embedded_fonts no)
